File: lumberjack.kicad_pcb (KiCad board)
At the start: 2 copper layers, 285.4 x 94.9 mm, 142 parts, among them J1 RJ45, U1 74HC14, U2 74HC14, U3 74HC14, U4 74HC14, U5 4021, U6 4021

Commit message: Couple of wires on the wrong side
Routing:
- net /R5.2: track 29.2 -> 36.5 mm
- net /R5.4: track 68.3 -> 71.7 mm
- net /R5.5: track 87.9 -> 89.1 mm
- net /R5.3: track 50.3 -> 51.1 mm
Changed lines of the file:
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@@
     (thickness 1.6)
     (drawings 144)
-    (tracks 1255)
+    (tracks 1253)
     (zones 0)
     (modules 142)
@@
   (segment (start 186.69 137.954) (end 183.356 134.62) (width 0.25) (layer B.Cu) (net 5))
   (segment (start 183.356 134.62) (end 177.8 134.62) (width 0.25) (layer B.Cu) (net 5))
-  (segment (start 196.215 137.954) (end 186.69 137.954) (width 0.25) (layer F.Cu) (net 5))
+  (segment (start 186.69 137.954) (end 196.215 137.954) (width 0.25) (layer B.Cu) (net 5))
   (segment (start 171.45 74.93) (end 169.9247 74.93) (width 0.25) (layer F.Cu) (net 6))
   (segment (start 154.94 69.85) (end 158.1174 69.85) (width 0.25) (layer F.Cu) (net 6))
@@
   (segment (start 177.8 118.11) (end 185.896 118.11) (width 0.25) (layer B.Cu) (net 76))
   (segment (start 185.896 118.11) (end 186.69 118.904) (width 0.25) (layer B.Cu) (net 76))
-  (segment (start 177.8 147.32) (end 178.9753 147.32) (width 0.25) (layer F.Cu) (net 77))
-  (segment (start 281.94 137.954) (end 278.0285 137.954) (width 0.25) (layer F.Cu) (net 77))
-  (segment (start 278.0285 137.954) (end 270.7118 145.2707) (width 0.25) (layer F.Cu) (net 77))
-  (segment (start 270.7118 145.2707) (end 181.0246 145.2707) (width 0.25) (layer F.Cu) (net 77))
-  (segment (start 181.0246 145.2707) (end 178.9753 147.32) (width 0.25) (layer F.Cu) (net 77))
-  (segment (start 262.89 137.954) (end 258.9785 137.954) (width 0.25) (layer F.Cu) (net 78))
-  (segment (start 258.9785 137.954) (end 252.1525 144.78) (width 0.25) (layer F.Cu) (net 78))
-  (segment (start 252.1525 144.78) (end 177.8 144.78) (width 0.25) (layer F.Cu) (net 78))
-  (segment (start 177.8 142.24) (end 178.9753 142.24) (width 0.25) (layer F.Cu) (net 79))
-  (segment (start 243.84 137.954) (end 239.9285 137.954) (width 0.25) (layer F.Cu) (net 79))
-  (segment (start 239.9285 137.954) (end 235.068 142.8145) (width 0.25) (layer F.Cu) (net 79))
-  (segment (start 235.068 142.8145) (end 179.5498 142.8145) (width 0.25) (layer F.Cu) (net 79))
-  (segment (start 179.5498 142.8145) (end 178.9753 142.24) (width 0.25) (layer F.Cu) (net 79))
-  (segment (start 177.8 139.7) (end 178.9753 139.7) (width 0.25) (layer B.Cu) (net 80))
-  (segment (start 224.79 137.954) (end 218.8726 137.954) (width 0.25) (layer B.Cu) (net 80))
-  (segment (start 218.8726 137.954) (end 213.9993 142.8273) (width 0.25) (layer B.Cu) (net 80))
-  (segment (start 213.9993 142.8273) (end 182.1026 142.8273) (width 0.25) (layer B.Cu) (net 80))
-  (segment (start 182.1026 142.8273) (end 178.9753 139.7) (width 0.25) (layer B.Cu) (net 80))
-  (segment (start 177.8 137.16) (end 178.9753 137.16) (width 0.25) (layer F.Cu) (net 81))
-  (segment (start 205.74 137.954) (end 202.565 137.954) (width 0.25) (layer F.Cu) (net 81))
-  (segment (start 202.565 137.954) (end 201.0946 136.4836) (width 0.25) (layer F.Cu) (net 81))
-  (segment (start 201.0946 136.4836) (end 195.1454 136.4836) (width 0.25) (layer F.Cu) (net 81))
-  (segment (start 195.1454 136.4836) (end 194.7101 136.9189) (width 0.25) (layer F.Cu) (net 81))
-  (segment (start 194.7101 136.9189) (end 187.9365 136.9189) (width 0.25) (layer F.Cu) (net 81))
-  (segment (start 187.9365 136.9189) (end 187.4966 136.479) (width 0.25) (layer F.Cu) (net 81))
-  (segment (start 187.4966 136.479) (end 179.6563 136.479) (width 0.25) (layer F.Cu) (net 81))
-  (segment (start 179.6563 136.479) (end 178.9753 137.16) (width 0.25) (layer F.Cu) (net 81))
+  (segment (start 177.8 147.32) (end 184.15 147.32) (width 0.25) (layer B.Cu) (net 77))
+  (segment (start 184.15 147.32) (end 186.182 145.288) (width 0.25) (layer B.Cu) (net 77))
+  (segment (start 280.323554 137.954) (end 281.94 137.954) (width 0.25) (layer B.Cu) (net 77))
+  (segment (start 272.989554 145.288) (end 280.323554 137.954) (width 0.25) (layer B.Cu) (net 77))
+  (segment (start 186.182 145.288) (end 272.989554 145.288) (width 0.25) (layer B.Cu) (net 77))
+  (segment (start 260.318 137.954) (end 262.89 137.954) (width 0.25) (layer B.Cu) (net 78))
+  (segment (start 259.334 138.938) (end 260.318 137.954) (width 0.25) (layer B.Cu) (net 78))
+  (segment (start 259.334 141.039666) (end 259.334 138.938) (width 0.25) (layer B.Cu) (net 78))
+  (segment (start 255.593666 144.78) (end 259.334 141.039666) (width 0.25) (layer B.Cu) (net 78))
+  (segment (start 177.8 144.78) (end 255.593666 144.78) (width 0.25) (layer B.Cu) (net 78))
+  (segment (start 179.832 144.272) (end 177.8 142.24) (width 0.25) (layer B.Cu) (net 79))
+  (segment (start 239.776 143.51) (end 239.014 144.272) (width 0.25) (layer B.Cu) (net 79))
+  (segment (start 239.776 139.7) (end 239.776 143.51) (width 0.25) (layer B.Cu) (net 79))
+  (segment (start 241.522 137.954) (end 239.776 139.7) (width 0.25) (layer B.Cu) (net 79))
+  (segment (start 239.014 144.272) (end 179.832 144.272) (width 0.25) (layer B.Cu) (net 79))
+  (segment (start 243.84 137.954) (end 241.522 137.954) (width 0.25) (layer B.Cu) (net 79))
+  (segment (start 181.864 143.764) (end 216.916 143.764) (width 0.25) (layer B.Cu) (net 80))
+  (segment (start 222.726 137.954) (end 224.79 137.954) (width 0.25) (layer B.Cu) (net 80))
+  (segment (start 216.916 143.764) (end 222.726 137.954) (width 0.25) (layer B.Cu) (net 80))
+  (segment (start 177.8 139.7) (end 181.864 143.764) (width 0.25) (layer B.Cu) (net 80))
+  (segment (start 206.756 138.97) (end 205.74 137.954) (width 0.25) (layer B.Cu) (net 81))
+  (segment (start 206.756 141.986) (end 206.756 138.97) (width 0.25) (layer B.Cu) (net 81))
+  (segment (start 205.486 143.256) (end 206.756 141.986) (width 0.25) (layer B.Cu) (net 81))
+  (segment (start 183.896 143.256) (end 205.486 143.256) (width 0.25) (layer B.Cu) (net 81))
+  (segment (start 177.8 137.16) (end 183.896 143.256) (width 0.25) (layer B.Cu) (net 81))
   (segment (start 132.08 85.09) (end 132.08 87.63) (width 0.25) (layer B.Cu) (net 82))
   (segment (start 151.13 95.25) (end 143.51 95.25) (width 0.25) (layer F.Cu) (net 83))

Commit message: With filled ground
Routing:
- net /BtnRightDebounced: track 31.3 -> 32.0 mm
- net +5V: vias 2 -> 0
- added copper zone on F.Cu, net GND
Changed lines of the file:
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@@
     (thickness 1.6)
     (drawings 144)
-    (tracks 1253)
+    (tracks 1248)
     (zones 0)
     (modules 142)
@@
   )
   (setup
-    (last_trace_width 0.25)
+    (last_trace_width 0.8)
     (user_trace_width 0.2)
     (user_trace_width 0.5)
@@
   (segment (start 147.588 101.092) (end 149.098 102.602) (width 0.8) (layer F.Cu) (net 1))
   (segment (start 146.304 101.092) (end 147.588 101.092) (width 0.8) (layer F.Cu) (net 1))
-  (via (at 146.812 85.598) (size 0.6) (drill 0.4) (layers F.Cu B.Cu) (net 1))
-  (segment (start 149.86 82.55) (end 146.812 85.598) (width 0.8) (layer B.Cu) (net 1))
-  (segment (start 151.13 82.55) (end 149.86 82.55) (width 0.8) (layer B.Cu) (net 1))
-  (via (at 146.812 89.154) (size 0.6) (drill 0.4) (layers F.Cu B.Cu) (net 1))
-  (segment (start 146.812 85.598) (end 146.812 89.154) (width 0.8) (layer F.Cu) (net 1))
-  (segment (start 146.812 100.584) (end 146.304 101.092) (width 0.8) (layer B.Cu) (net 1))
-  (segment (start 146.812 89.154) (end 146.812 100.584) (width 0.8) (layer B.Cu) (net 1))
   (segment (start 129.54 67.31) (end 127 64.77) (width 0.8) (layer B.Cu) (net 1))
   (segment (start 129.54 76.708) (end 129.54 67.31) (width 0.8) (layer B.Cu) (net 1))
   (segment (start 132.08 79.248) (end 129.54 76.708) (width 0.8) (layer B.Cu) (net 1))
+  (segment (start 146.812 100.584) (end 146.304 101.092) (width 0.8) (layer B.Cu) (net 1))
+  (segment (start 146.812 85.598) (end 146.812 100.584) (width 0.8) (layer B.Cu) (net 1))
+  (segment (start 149.86 82.55) (end 146.812 85.598) (width 0.8) (layer B.Cu) (net 1))
+  (segment (start 151.13 82.55) (end 149.86 82.55) (width 0.8) (layer B.Cu) (net 1))
   (segment (start 134.62 138.8702) (end 134.62 139.66) (width 0.25) (layer F.Cu) (net 2))
   (segment (start 122.3951 133.1289) (end 122.936 132.588) (width 0.8) (layer F.Cu) (net 2))
@@
   (segment (start 151.638 85.09) (end 152.908 86.36) (width 0.25) (layer F.Cu) (net 102))
   (segment (start 151.13 85.09) (end 151.638 85.09) (width 0.25) (layer F.Cu) (net 102))
-  (segment (start 145.0353 90.17) (end 145.0353 89.1214) (width 0.25) (layer B.Cu) (net 103))
-  (segment (start 145.0353 89.1214) (end 150.3367 83.82) (width 0.25) (layer B.Cu) (net 103))
-  (segment (start 150.3367 83.82) (end 151.9156 83.82) (width 0.25) (layer B.Cu) (net 103))
-  (segment (start 151.9156 83.82) (end 152.8229 82.9127) (width 0.25) (layer B.Cu) (net 103))
-  (segment (start 152.8229 82.9127) (end 152.8229 82.1715) (width 0.25) (layer B.Cu) (net 103))
-  (segment (start 143.51 90.17) (end 145.0353 90.17) (width 0.25) (layer B.Cu) (net 103))
   (segment (start 163.83 72.39) (end 163.322 72.39) (width 0.25) (layer B.Cu) (net 103))
   (segment (start 163.322 72.39) (end 161.544 74.168) (width 0.25) (layer B.Cu) (net 103))
-  (segment (start 152.8229 82.1715) (end 154.0732 80.9212) (width 0.25) (layer B.Cu) (net 103))
-  (segment (start 154.0732 80.9212) (end 159.193394 80.9212) (width 0.25) (layer B.Cu) (net 103))
-  (segment (start 161.544 78.570594) (end 161.544 74.168) (width 0.25) (layer B.Cu) (net 103))
-  (segment (start 159.193394 80.9212) (end 161.544 78.570594) (width 0.25) (layer B.Cu) (net 103))
+  (segment (start 146.05 85.467394) (end 146.05 84.582) (width 0.25) (layer B.Cu) (net 103))
+  (segment (start 146.05 84.582) (end 152.71199 77.92001) (width 0.25) (layer B.Cu) (net 103))
+  (segment (start 145.0353 86.482094) (end 146.05 85.467394) (width 0.25) (layer B.Cu) (net 103))
+  (segment (start 145.0353 90.17) (end 145.0353 86.482094) (width 0.25) (layer B.Cu) (net 103))
+  (segment (start 143.51 90.17) (end 145.0353 90.17) (width 0.25) (layer B.Cu) (net 103))
+  (segment (start 161.544 74.168) (end 161.544 76.962) (width 0.25) (layer B.Cu) (net 103))
+  (segment (start 160.58599 77.92001) (end 152.71199 77.92001) (width 0.25) (layer B.Cu) (net 103))
+  (segment (start 161.544 76.962) (end 160.58599 77.92001) (width 0.25) (layer B.Cu) (net 103))
   (segment (start 171.45 64.77) (end 169.9247 64.77) (width 0.25) (layer B.Cu) (net 104))
   (segment (start 151.13 97.79) (end 152.6553 97.79) (width 0.25) (layer B.Cu) (net 104))
@@
   (segment (start 132.08 69.85) (end 132.08 72.39) (width 0.25) (layer F.Cu) (net 124))
   (segment (start 127 58.42) (end 127 57.15) (width 0.25) (layer F.Cu) (net 124))
+  (zone (net 2) (net_name GND) (layer F.Cu) (hatch edge 0.508)
+    (connect_pads (clearance 0.508))
+    (min_thickness 0.254)
+    (fill yes (arc_segments 32) (thermal_gap 0.508) (thermal_bridge_width 0.508))
+    (polygon
+      (pts
+        (xy 292.608 147.32) (xy 12.192 147.32) (xy 12.192 57.404) (xy 292.608 57.404)
+      )
+    )
+  )
 )

Commit message: Finished V1 PCB?
Routing:
- net GND: track 2311.0 -> 2336.0 mm, vias 0 -> 3
- added copper zone on B.Cu, net +5V
Changed lines of the file:
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@@
   (general
     (thickness 1.6)
-    (drawings 144)
-    (tracks 1248)
+    (drawings 160)
+    (tracks 1260)
     (zones 0)
     (modules 142)
@@
   )
   (setup
-    (last_trace_width 0.8)
+    (last_trace_width 0.25)
     (user_trace_width 0.2)
     (user_trace_width 0.5)
@@
       (net 2 GND))
   )
-  (gr_text > (at 177.8 65.024 180) (layer F.SilkS)
+  (gr_text > (at 175.768 133.858 180) (layer F.SilkS)
+    (effects (font (size 1.5 1.5) (thickness 0.3)))
+  )
+  (gr_text > (at 175.768 130.81) (layer F.SilkS)
+    (effects (font (size 1.5 1.5) (thickness 0.3)))
+  )
+  (gr_text > (at 175.768 118.364 180) (layer F.SilkS)
+    (effects (font (size 1.5 1.5) (thickness 0.3)))
+  )
+  (gr_text > (at 175.514 101.854 180) (layer F.SilkS)
+    (effects (font (size 1.5 1.5) (thickness 0.3)))
+  )
+  (gr_text > (at 175.768 114.3) (layer F.SilkS)
+    (effects (font (size 1.5 1.5) (thickness 0.3)))
+  )
+  (gr_text > (at 176.022 96.52) (layer F.SilkS)
+    (effects (font (size 1.5 1.5) (thickness 0.3)))
+  )
+  (gr_text > (at 176.022 83.82 180) (layer F.SilkS)
+    (effects (font (size 1.5 1.5) (thickness 0.3)))
+  )
+  (gr_text > (at 175.768 80.01) (layer F.SilkS)
+    (effects (font (size 1.5 1.5) (thickness 0.3)))
+  )
+  (gr_text > (at 129.286 81.28) (layer F.SilkS)
+    (effects (font (size 1.5 1.5) (thickness 0.3)))
+  )
+  (gr_text > (at 129.286 97.79) (layer F.SilkS)
+    (effects (font (size 1.5 1.5) (thickness 0.3)))
+  )
+  (gr_text > (at 129.032 114.3) (layer F.SilkS)
+    (effects (font (size 1.5 1.5) (thickness 0.3)))
+  )
+  (gr_text > (at 128.524 133.096 180) (layer F.SilkS)
+    (effects (font (size 1.5 1.5) (thickness 0.3)))
+  )
+  (gr_text > (at 129.032 118.364 180) (layer F.SilkS)
+    (effects (font (size 1.5 1.5) (thickness 0.3)))
+  )
+  (gr_text > (at 129.286 101.854 180) (layer F.SilkS)
+    (effects (font (size 1.5 1.5) (thickness 0.3)))
+  )
+  (gr_text > (at 129.286 85.09 180) (layer F.SilkS)
+    (effects (font (size 1.5 1.5) (thickness 0.3)))
+  )
+  (gr_text > (at 129.286 68.58 180) (layer F.SilkS)
+    (effects (font (size 1.5 1.5) (thickness 0.3)))
+  )
+  (gr_text > (at 175.768 67.564 180) (layer F.SilkS)
     (effects (font (size 1.5 1.5) (thickness 0.3)))
   )
@@
   (segment (start 170.688 77.216) (end 172.172 77.216) (width 0.8) (layer F.Cu) (net 2))
   (segment (start 168.402 74.93) (end 170.688 77.216) (width 0.8) (layer F.Cu) (net 2))
-  (segment (start 163.83 74.93) (end 168.402 74.93) (width 0.8) (layer F.Cu) (net 2))
   (segment (start 170.18 82.55) (end 172.68 80.05) (width 0.8) (layer F.Cu) (net 2))
   (segment (start 172.68 80.05) (end 172.68 79.248) (width 0.8) (layer F.Cu) (net 2))
@@
   (segment (start 128.288902 133.1289) (end 128.778 133.617998) (width 0.8) (layer F.Cu) (net 2))
   (segment (start 127.9831 133.1289) (end 128.288902 133.1289) (width 0.8) (layer F.Cu) (net 2))
+  (via (at 168.402 58.928) (size 0.6) (drill 0.4) (layers F.Cu B.Cu) (net 2))
+  (segment (start 168.76501 58.56499) (end 168.402 58.928) (width 0.25) (layer B.Cu) (net 2))
+  (segment (start 174.42899 58.56499) (end 168.76501 58.56499) (width 0.25) (layer B.Cu) (net 2))
+  (segment (start 175.768 59.904) (end 174.42899 58.56499) (width 0.25) (layer B.Cu) (net 2))
+  (via (at 166.37 62.992) (size 0.6) (drill 0.4) (layers F.Cu B.Cu) (net 2))
+  (segment (start 166.37 60.96) (end 166.37 62.992) (width 0.25) (layer F.Cu) (net 2))
+  (segment (start 168.402 58.928) (end 166.37 60.96) (width 0.25) (layer F.Cu) (net 2))
+  (segment (start 166.37 62.992) (end 166.624 63.246) (width 0.25) (layer B.Cu) (net 2))
+  (via (at 166.624 74.422) (size 0.6) (drill 0.4) (layers F.Cu B.Cu) (net 2))
+  (segment (start 166.624 63.246) (end 166.624 74.422) (width 0.25) (layer B.Cu) (net 2))
+  (segment (start 166.624 74.422) (end 166.624 74.93) (width 0.25) (layer F.Cu) (net 2))
+  (segment (start 166.624 74.93) (end 168.402 74.93) (width 0.8) (layer F.Cu) (net 2))
+  (segment (start 163.83 74.93) (end 166.624 74.93) (width 0.8) (layer F.Cu) (net 2))
   (segment (start 166.116 102.616) (end 156.464 102.616) (width 0.8) (layer F.Cu) (net 3))
   (segment (start 110.49 137.954) (end 110.49 138.43) (width 0.2) (layer B.Cu) (net 4))
@@
   (segment (start 127 59.69) (end 132.08 64.77) (width 0.25) (layer F.Cu) (net 124))
   (segment (start 127 58.42) (end 127 59.69) (width 0.25) (layer F.Cu) (net 124))
-  (segment (start 132.08 64.77) (end 132.08 67.31) (width 0.25) (layer F.Cu) (net 124))
-  (segment (start 132.08 67.31) (end 132.08 69.85) (width 0.25) (layer F.Cu) (net 124))
-  (segment (start 132.08 69.85) (end 132.08 72.39) (width 0.25) (layer F.Cu) (net 124))
   (segment (start 127 58.42) (end 127 57.15) (width 0.25) (layer F.Cu) (net 124))
+  (segment (start 132.08 64.77) (end 132.08 67.31) (width 0.25) (layer B.Cu) (net 124))
+  (segment (start 132.08 67.31) (end 132.08 69.85) (width 0.25) (layer B.Cu) (net 124))
+  (segment (start 132.08 69.85) (end 132.08 72.39) (width 0.25) (layer B.Cu) (net 124))
   (zone (net 2) (net_name GND) (layer F.Cu) (hatch edge 0.508)
     (connect_pads (clearance 0.508))
@@
       )
     )
+  )
+  (zone (net 1) (net_name +5V) (layer B.Cu) (hatch edge 0.508)
+    (connect_pads (clearance 0.508))
+    (min_thickness 0.254)
+    (fill yes (arc_segments 32) (thermal_gap 0.508) (thermal_bridge_width 0.508))
+    (polygon
+      (pts
+        (xy 181.102 147.32) (xy 123.698 147.32) (xy 123.698 57.404) (xy 181.102 57.404)
+      )
+    )
